File: kicad/stm8l_test.kicad_pcb (KiCad board)
At the start: 2 copper layers, 26 parts, among them J1 Conn_01x04, J2 Conn_01x02, Q1 2N7002, SW1 SW_Push, SW2 prog_sw, SW3 Rotary_Encoder_Switch, U2 STM8L101F3P, U3 BD70522GUL-E2

Commit message: Pdb work, schema done
Parts:
- removed J2: Conn_01x02, TerminalBlock_Phoenix:TerminalBlock_Phoenix_PT-1,5-2-5.0-H_1x02_P5.00mm_Horizontal
- removed R8: 180, Resistor_SMD:R_0603_1608Metric_Pad1.05x0.95mm_HandSolder
- removed U3: BD70522GUL-E2, good_things:BGA-9_3x3_1.76x1.56mm
- added BT1: Battery_Cell, Battery:BatteryHolder_Keystone_3002_1x2032, B.Cu at (96.0, 76.5)
- added D1: D_Small, Diode_SMD:D_1210_3225Metric_Pad1.42x2.65mm_HandSolder, F.Cu at (74.0, 94.0)
- added D11: VLMO30L1M2-GS18, LED_SMD:LED_PLCC-2, F.Cu at (134.6, 80.0)
- added D12: VLMO30L1M2-GS18, LED_SMD:LED_PLCC-2, F.Cu at (136.5, 83.7)
- added D13: VLMO30L1M2-GS18, LED_SMD:LED_PLCC-2, F.Cu at (138.0, 87.6)
- added D14: VLMO30L1M2-GS18, LED_SMD:LED_PLCC-2, F.Cu at (139.1, 91.7)
- added D15: VLMO30L1M2-GS18, LED_SMD:LED_PLCC-2, F.Cu at (139.8, 95.8)
- added D16: VLMO30L1M2-GS18, LED_SMD:LED_PLCC-2, F.Cu at (140.0, 100.0)
- added D17: VLMO30L1M2-GS18, LED_SMD:LED_PLCC-2, F.Cu at (139.8, 104.2)
- added D18: VLMO30L1M2-GS18, LED_SMD:LED_PLCC-2, F.Cu at (139.1, 108.3)
- added D19: VLMO30L1M2-GS18, LED_SMD:LED_PLCC-2, F.Cu at (138.0, 112.4)
- added D20: VLMO30L1M2-GS18, LED_SMD:LED_PLCC-2, F.Cu at (134.6, 120.0)
- added D21: VLMO30L1M2-GS18, LED_SMD:LED_PLCC-2, F.Cu at (129.7, 126.8)
- added D22: VLMO30L1M2-GS18, LED_SMD:LED_PLCC-2, F.Cu at (123.5, 132.4)
- added D23: VLMO30L1M2-GS18, LED_SMD:LED_PLCC-2, F.Cu at (116.3, 136.5)
- added D24: VLMO30L1M2-GS18, LED_SMD:LED_PLCC-2, F.Cu at (108.3, 139.1)
- added D25: VLMO30L1M2-GS18, LED_SMD:LED_PLCC-2, F.Cu at (100.0, 140.0)
- added D26: VLMO30L1M2-GS18, LED_SMD:LED_PLCC-2, F.Cu at (80.0, 134.6)
- added D27: VLMO30L1M2-GS18, LED_SMD:LED_PLCC-2, F.Cu at (65.4, 120.0)
- added D28: VLMO30L1M2-GS18, LED_SMD:LED_PLCC-2, F.Cu at (60.0, 100.0)
- added D29: VLMO30L1M2-GS18, LED_SMD:LED_PLCC-2, F.Cu at (65.4, 80.0)
- added D30: VLMO30L1M2-GS18, LED_SMD:LED_PLCC-2, F.Cu at (80.0, 65.4)
- added D31: VLMO30L1M2-GS18, LED_SMD:LED_PLCC-2, F.Cu at (100.0, 60.0)
- added F1: 500ma, Fuse:Fuse_1206_3216Metric_Pad1.42x1.75mm_HandSolder, F.Cu at (112.2, 97.0)
- added H1: MountingHole, MountingHole:MountingHole_2.7mm_M2.5, F.Cu at (266.5, 23.0)
- added H2: MountingHole, MountingHole:MountingHole_2.7mm_M2.5, F.Cu at (266.5, 29.9)
- added H3: MountingHole, MountingHole:MountingHole_2.7mm_M2.5, F.Cu at (273.4, 23.0)
- added H4: MountingHole, MountingHole:MountingHole_2.7mm_M2.5, F.Cu at (273.4, 29.9)
- added Q2: 2N7002, Package_TO_SOT_SMD:SOT-23, F.Cu at (81.5, 92.7)
- added Q3: SI2365EDS-T1-GE3, Package_TO_SOT_SMD:SOT-23_Handsoldering, F.Cu at (152.5, 108.5)
- added Q4: SI2365EDS-T1-GE3, Package_TO_SOT_SMD:SOT-23_Handsoldering, F.Cu at (228.0, 67.5)
- added Q5: SI2365EDS-T1-GE3, Package_TO_SOT_SMD:SOT-23_Handsoldering, F.Cu at (151.8, 44.5)
- added Q6: SI2365EDS-T1-GE3, Package_TO_SOT_SMD:SOT-23_Handsoldering, F.Cu at (174.5, 36.5)
- added Q7: SI2365EDS-T1-GE3, Package_TO_SOT_SMD:SOT-23_Handsoldering, F.Cu at (199.0, 140.0)
- added Q8: SI2365EDS-T1-GE3, Package_TO_SOT_SMD:SOT-23_Handsoldering, F.Cu at (248.1, 87.3)
- added R3: 1k, Resistor_SMD:R_0603_1608Metric_Pad1.05x0.95mm_HandSolder, F.Cu at (74.1, 89.0)
- added R4: 180, Resistor_SMD:R_0603_1608Metric_Pad1.05x0.95mm_HandSolder, F.Cu at (300.3, 147.7)
- added U1: BD70522GUL-E2, good_things:BGA-9_3x3_1.76x1.56mm, F.Cu at (120.6, 103.4)
- C1: value 10u -> 22u; footprint Capacitor_SMD:C_0805_2012Metric_Pad1.15x1.40mm_HandSolder -> Capacitor_SMD:C_0603_1608Metric_Pad1.05x0.95mm_HandSolder
- C2: value 100n -> 22u
- C3: footprint Capacitor_SMD:C_0805_2012Metric_Pad1.15x1.40mm_HandSolder -> Capacitor_SMD:C_0603_1608Metric_Pad1.05x0.95mm_HandSolder
- C4: value 22u -> 100n; footprint Capacitor_SMD:C_0805_2012Metric_Pad1.15x1.40mm_HandSolder -> Capacitor_SMD:C_0603_1608Metric_Pad1.05x0.95mm_HandSolder
- D10, D2, D3, D4, D5, D7, D8, D9: value red -> VLMO30L1M2-GS18; footprint LED_SMD:LED_1206_3216Metric_Pad1.42x1.75mm_HandSolder -> LED_SMD:LED_PLCC-2
- D6: value D_Small -> VLMO30L1M2-GS18; footprint Diode_SMD:D_1210_3225Metric_Pad1.42x2.65mm_HandSolder -> LED_SMD:LED_PLCC-2
- J1: footprint Connector_PinHeader_2.54mm:PinHeader_1x04_P2.54mm_Vertical -> good_things:TSM-104-01-L-SH
- Q1: value 2N7002 -> SI2365EDS-T1-GE3; footprint Package_TO_SOT_SMD:SOT-23 -> Package_TO_SOT_SMD:SOT-23_Handsoldering
- R1: value 10k -> 100k
- R2: value 1k -> 100k
- SW1: value SW_Push -> prog_sw; footprint Button_Switch_THT:SW_PUSH_6mm -> good_things:TSM-103-01-l_SH
- SW2: value prog_sw -> SW_Push; footprint Connector_PinSocket_2.54mm:PinSocket_1x03_P2.54mm_Vertical -> good_things:push_sw_purple
- moved C2 279.5 mm to (308.4, 142.9), turned to 0 degrees
- moved R2 267.9 mm to (295.9, 147.7), turned to 0 degrees
- moved U2 234.8 mm to (100.0, 116.0)
- moved SW3 230.6 mm to (92.5, 102.5)
- moved L1 226.3 mm to (115.5, 106.1), turned to 270 degrees
- moved C3 217.3 mm to (121.9, 106.0)
- moved C1 215.9 mm to (120.6, 101.4), turned to 0 degrees
- moved BZ1 215.3 mm to (74.0, 91.0), turned to 0 degrees
- moved R1 208.5 mm to (112.8, 100.0), turned to 180 degrees
- moved Q1 205.7 mm to (116.7, 98.5), turned to 90 degrees
- moved SW2 203.4 mm to (114.0, 91.0), turned to 0 degrees
- moved J1 195.3 mm to (126.0, 85.0), turned to 0 degrees
- moved D10 185.0 mm to (132.4, 76.5), turned to 36 degrees
- moved SW1 184.5 mm to (117.5, 82.2), turned to 180 degrees
- moved D9 182.2 mm to (129.7, 73.2), turned to 42 degrees
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Connections:
- net swim_data renamed pa0
- BZ1 pad 1: vcc -> vbat
- C1 pad 1: vbat -> vcc
- C3 pad 1: vcc -> vled
- C4 pad 1: 1v8 -> vcc
- D10 pad 1: GND -> c3
- D10 pad 2: b7 -> Net-(D10-Pad2)
- D2 pad 1: GND -> c4
- D2 pad 2: b0 -> Net-(D14-Pad2)
- D3 pad 1: GND -> c4
- D3 pad 2: b1 -> Net-(D15-Pad2)
- D4 pad 1: GND -> c4
- D4 pad 2: b2 -> Net-(D10-Pad2)
- D5 pad 1: GND -> c4
- D5 pad 2: b3 -> Net-(D11-Pad2)
- D6 pad 1: vcc -> c4
- D6 pad 2: Net-(BZ1-Pad2) -> Net-(D12-Pad2)
- D7 pad 1: GND -> c4
- D7 pad 2: b4 -> Net-(D13-Pad2)
- D8 pad 1: GND -> c3
- D8 pad 2: b5 -> Net-(D14-Pad2)
- D9 pad 1: GND -> c3
- D9 pad 2: b6 -> Net-(D15-Pad2)
- L1 pad 2: 1v8 -> vled
- Q1 pad 2: GND -> vcc
- Q1 pad 3: Net-(BZ1-Pad2) -> Net-(F1-Pad2)
- R1 pad 1: vcc -> Net-(Q1-Pad1)
- R1 pad 2: rst -> GND
- R2 pad 2: Net-(BZ1-Pad2) -> encoder_sw
- SW1 pad 1: GND -> prog_v
- SW1 pad 2: rst -> Net-(F1-Pad1)
- SW2 pad 1: prog_v -> GND
- SW2 pad 2: vcc -> rst
- SW3 pad S1: vcc -> encoder_sw
- SW3 pad S2: encoder_sw -> GND
- U2 pad 1: (no net) -> c3
- U2 pad 10: b0 -> a0
- U2 pad 11: b1 -> a1
- U2 pad 12: b2 -> a2
- U2 pad 13: b3 -> a3
- U2 pad 14: b4 -> a4
- U2 pad 15: b5 -> a5
- U2 pad 16: b6 -> encoder_sw
- U2 pad 17: b7 -> led_enable
- U2 pad 18: encoder_sw -> c0
- U2 pad 19: encoder_a -> c1
- U2 pad 2: (no net) -> c4
- U2 pad 20: encoder_b -> c2
- U2 pad 5: (no net) -> encoder_b
- U2 pad 6: (no net) -> encoder_a
Routing:
- net vcc: track 75.0 -> 0.00 mm
- net rst: track 30.1 -> 0.00 mm
- net b7: track 27.3 -> 0.00 mm
- net 1v8: track 26.1 -> 0.00 mm
- net b6: track 25.2 -> 0.00 mm
- net b0: track 25.1 -> 0.00 mm
- net encoder_sw: track 23.5 -> 0.00 mm
- net b5: track 22.0 -> 0.00 mm
- net vbat: track 20.3 -> 0.00 mm
- net b4: track 19.3 -> 0.00 mm
- net b3: track 16.7 -> 0.00 mm
- net b2: track 13.8 -> 0.00 mm
- net GND: track 14.6 -> 1.00 mm
- net pa0: track 11.8 -> 0.00 mm
- net b1: track 11.0 -> 0.00 mm
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- removed copper zone on F.Cu, net GND
Other:
- board outline added: 90 x 90 mm
- net class Default: via_dia 1.5 -> 0.8
- net class smool conv removed
- board text removed: "stm8 dev V1 Anton Lööf"

Commit message: Place components and initial routing
Parts:
- removed C2: 22u, Capacitor_SMD:C_0603_1608Metric_Pad1.05x0.95mm_HandSolder
- D10, D11, D12, D13, D14, D15, D16, D17, D18, D19, D2, D20, D21, D22, D23, D24, D25, D26, D27, D28, D29, D3, D30, D31, D4, D5, D6, D7, D8, D9: value VLMO30L1M2-GS18 -> TLMS1000-GS08; footprint LED_SMD:LED_PLCC-2 -> LED_SMD:LED_0603_1608Metric_Pad1.05x0.95mm_HandSolder
- moved H3 147.5 mm to (153.4, 108.7)
- moved H2 144.5 mm to (134.6, 88.9)
- moved R4 135.5 mm to (171.5, 105.6), turned to 90 degrees
- moved H1 134.3 mm to (148.7, 87.4)
- moved R2 133.6 mm to (175.2, 90.5), turned to 180 degrees
- moved H4 111.0 mm to (177.1, 85.1)
- moved R3 90.2 mm to (161.7, 110.5)
- moved BZ1 89.6 mm to (161.8, 108.8)
- moved D1 88.6 mm to (161.8, 106.0)
- moved Q2 87.6 mm to (168.1, 105.5), turned to 180 degrees
- moved Q6 84.6 mm to (170.3, 121.0)
- moved U2 82.6 mm to (180.1, 95.5), turned to 270 degrees
- moved Q5 76.3 mm to (174.1, 117.5)
- moved D28 71.9 mm to (131.8, 96.5), turned to 0 degrees
- moved D27 71.1 mm to (136.1, 112.5), turned to 30 degrees
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Connections:
- U1 pad C1: (no net) -> Net-(U1-PadC1)
- U2 pad 5: encoder_b -> encoder_a
- U2 pad 6: encoder_a -> encoder_b
Routing:
- net Net-(D10-Pad2): track 0.00 -> 158.0 mm, vias 0 -> 8
- net c0: track 0.00 -> 154.8 mm, vias 0 -> 2
- net Net-(D15-Pad2): track 0.00 -> 146.6 mm, vias 0 -> 9
- net Net-(D11-Pad2): track 0.00 -> 145.8 mm, vias 0 -> 8
- net Net-(D14-Pad2): track 0.00 -> 130.0 mm, vias 0 -> 8
- net Net-(D12-Pad2): track 0.00 -> 127.8 mm, vias 0 -> 8
- net Net-(D13-Pad2): track 0.00 -> 118.0 mm, vias 0 -> 8
- net vbat: track 0.00 -> 72.0 mm, vias 0 -> 2
- net rst: track 0.00 -> 62.6 mm, vias 0 -> 1
- net c1: track 0.00 -> 61.5 mm, vias 0 -> 2
- net vcc: track 0.00 -> 52.4 mm, vias 0 -> 3
- net Net-(F1-Pad1): track 0.00 -> 43.7 mm, vias 0 -> 8
- net vled: track 0.00 -> 43.5 mm
- net c4: track 0.00 -> 42.5 mm
- net pa0: track 0.00 -> 42.4 mm, vias 0 -> 1
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- added copper zone on B.Cu, net Net-(F1-Pad1)
- added copper zone on F.Cu, net Net-(F1-Pad1)
Other:
- board size 90 x 90 mm -> 72 x 72 mm

Commit message: PCB rev1 ordered
Parts:
- moved H3 17.0 mm to (170.3, 110.2)
- moved SW1 6.47 mm to (140.9, 87.7), turned to 180 degrees
- moved F1 5.92 mm to (147.6, 114.3)
- moved SW2 3.60 mm to (139.0, 102.1)
- moved J1 1.04 mm to (149.1, 92.7)
- moved C3 0.40 mm to (161.6, 114.0)
Routing:
- net prog_v: track 22.8 -> 2.97 mm
- net vbat: track 72.0 -> 84.2 mm
- net led_enable: track 39.9 -> 49.1 mm
- net pa0: track 42.4 -> 48.2 mm
- net Net-(F1-Pad1): track 43.7 -> 37.9 mm, vias 8 -> 7
- net Net-(F1-Pad2): track 8.41 -> 3.41 mm
- net rst: track 62.6 -> 66.7 mm
- net vcc: track 52.4 -> 55.9 mm
- net GND: track 8.94 -> 6.91 mm, vias 1 -> 0
- net vled: track 43.5 -> 44.2 mm
- added copper zone on B.Cu, net GND
- added copper zone on F.Cu, net GND
Other:
- board size 72 x 72 mm -> 70 x 70 mm
- rule pad_to_mask_clearance: 0.051 -> 0
- board text added: "3v3 pa0 gnd rst"
- board text added: "EggTimer V1 Anton Lööf 2021"
- board text added: "JLCJLCJLCJLC"
- board text added: "bat + prog"
