File: eggtimer_pcb/eggtimer_pcb.sch (KiCad schematic (older format))
At the start: 24 parts

Commit message: Schema is done
some layout work
Parts:
- added BZ1: Buzzer, good_things:buzzer_d14_p5, symbol Device:Buzzer
- added D1: RSX301L-30TE25, good_things:smd_diode_sod_106, symbol Device:D_Small
- added D10, D11, D12, D13, D14, D15, D16, D17, D18, D19, D2, D20, D21, D22, D23, D24, D25, D26, D27, D28, D29, D3, D30, D31, D32, D33, D34, D35, D36, D37, D4, D5, D6, D7, D8, D9: TLMS1000-GS08, LED_SMD:LED_0603_1608Metric_Pad1.05x0.95mm_HandSolder, symbol Device:LED
- added H1, H2, H3, H4: MountingHole_Pad, MountingHole:MountingHole_2.7mm_M2.5_DIN965_Pad, symbol Mechanical:MountingHole_Pad
- added JP1: power_bypass, Jumper:SolderJumper-2_P1.3mm_Open_TrianglePad1.0x1.5mm, symbol Jumper:SolderJumper_2_Open
- added Q1, Q2, Q3, Q4, Q5, Q6: CPH3350-TL-W, Package_TO_SOT_SMD:SOT-23_Handsoldering, symbol Device:Q_PMOS_GSD
- added Q10: 2N7002P,215, Package_TO_SOT_SMD:SOT-23_Handsoldering, symbol Device:Q_NMOS_GSD
- added R1, R3, R5, R6, R7, R8: 200, Resistor_SMD:R_0603_1608Metric_Pad0.98x0.95mm_HandSolder, symbol Device:R_Small
- added R11: 1k, Resistor_SMD:R_0603_1608Metric_Pad0.98x0.95mm_HandSolder, symbol Device:R_Small
- added R12: r_sense, Resistor_SMD:R_0603_1608Metric_Pad0.98x0.95mm_HandSolder, symbol Device:R_Small
- added TP2: debug_v, TestPoint:TestPoint_Pad_D1.5mm, symbol Connector:TestPoint
- added TP3: GND, TestPoint:TestPoint_Pad_D1.5mm, symbol Connector:TestPoint
- BT1, BT2: renamed from BT?; footprint (none) -> Battery:BatteryHolder_Keystone_2466_1xAAA
- C1, C2, C3, C4, C5, C6, C7, C8: renamed from C?; footprint (none) -> Capacitor_SMD:C_0603_1608Metric
- J1: renamed from J?; footprint (none) -> Connector_PinHeader_2.54mm:PinHeader_1x03_P2.54mm_Vertical
- L1: renamed from L?; value 1u5 -> 2u2; footprint (none) -> Inductor_SMD:L_Wuerth_MAPI-2010
- Q7, Q8, Q9: renamed from Q?; footprint (none) -> Package_TO_SOT_SMD:SOT-23_Handsoldering
- R2: renamed from R?; value 100k -> 1M; footprint (none) -> Resistor_SMD:R_0603_1608Metric_Pad0.98x0.95mm_HandSolder
- R4, R9: renamed from R?; footprint (none) -> Resistor_SMD:R_0603_1608Metric_Pad0.98x0.95mm_HandSolder
- SW1: renamed from SW?; footprint (none) -> Rotary_Encoder:RotaryEncoder_Alps_EC11E-Switch_Vertical_H20mm
- SW2: renamed from SW?; footprint (none) -> good_things:push_sw_purple
- TP1: renamed from TP?; footprint (none) -> TestPoint:TestPoint_Pad_D2.0mm
- U1: renamed from U?; footprint (none) -> good_things:BGA-9_3x3_1.76x1.56mm
- U2: renamed from U?; footprint (none) -> Package_DFN_QFN:QFN-28_4x4mm_P0.5mm
- Y1: renamed from Y?; footprint (none) -> Crystal:Crystal_Round_D3.0mm_Vertical
Connections:
- net 2v_led: now also Q1.2 (S), Q2.2 (S), Q3.2 (S), Q4.2 (S), Q5.2 (S), Q6.2 (S)
- net GND: now also H1.1, H2.1, H3.1, H4.1, Q10.2 (S), TP3.1
- net encoder_a: now also U2.18 (PA11); no longer U2.6 (PA0)
- net encoder_b: now also U2.19 (PA12); no longer U2.7 (PA1)
- net v_bat: now also R12.2, TP2.1; no longer Q7.3 (D), R2.2
- net vcc: now also BZ1.1 (-), D1.1 (K), JP1.2 (B), R11.1
- net led_c4: now reaches U2.10 (PA4)
- net led_c4: now also R7.1
- net led_c3: now reaches U2.11 (PA5)
- net led_c3: now also R6.1
- net led_c2: now reaches U2.12 (PA6)
- net led_c2: now also R5.1
- net led_c1: now reaches U2.13 (PA7)
- net led_c1: now also R3.1
- net led_c0: now reaches U2.14 (PB0)
- net led_c0: now also R1.1
- net buzzer_ctrl: now reaches U2.16 (PA8)
- net buzzer_ctrl: now also Q10.1 (G)
- net led_a0: now reaches U2.23 (PB3)
- net led_a0: now also Q1.1 (G)
- net led_a1: now reaches U2.24 (PB4)
- net led_a1: now also Q2.1 (G)
- net led_a2: now reaches U2.25 (PB5)
- net led_a2: now also Q3.1 (G)
- net led_a3: now reaches U2.26 (PB6)
- net led_a3: now also Q4.1 (G)
- net led_a4: now reaches U2.27 (PB7)
- net led_a4: now also Q5.1 (G)
- net led_a5: now reaches U2.28 (PB8)
- net led_a5: now also Q6.1 (G)
- net led_c5: now reaches U2.9 (PA3)
- net led_c5: now also R8.1
- net v_bat_prot: now reaches Q7.2 (S), Q8.2 (S), SW1.S1
- net v_bat_prot: now also R2.2, JP1.1 (A)
- net bat_center: now reaches BT1.2 (-), BT2.1 (+)
- net power_on: now reaches Q8.1 (G), Q9.3 (D), R2.1
- net vled_sw: now reaches L1.2, U1.A2 (lx)
- new net: D10.1 (K), D11.1 (K), D12.1 (K), D13.1 (K), D8.1 (K), D9.1 (K), R3.2
- new net: D14.2 (A), D2.2 (A), D20.2 (A), D26.2 (A), D32.2 (A), D8.2 (A), Q1.3 (D)
- new net: D14.1 (K), D15.1 (K), D16.1 (K), D17.1 (K), D18.1 (K), D19.1 (K), R5.2
- new net: D20.1 (K), D21.1 (K), D22.1 (K), D23.1 (K), D24.1 (K), D25.1 (K), R6.2
- new net: D26.1 (K), D27.1 (K), D28.1 (K), D29.1 (K), D30.1 (K), D31.1 (K), R7.2
- new net: D32.1 (K), D33.1 (K), D34.1 (K), D35.1 (K), D36.1 (K), D37.1 (K), R8.2
- new net: D2.1 (K), D3.1 (K), D4.1 (K), D5.1 (K), D6.1 (K), D7.1 (K), R1.2
- new net: D15.2 (A), D21.2 (A), D27.2 (A), D3.2 (A), D33.2 (A), D9.2 (A), Q2.3 (D)
- new net: D10.2 (A), D16.2 (A), D22.2 (A), D28.2 (A), D34.2 (A), D4.2 (A), Q3.3 (D)
- new net: D11.2 (A), D17.2 (A), D23.2 (A), D29.2 (A), D35.2 (A), D5.2 (A), Q4.3 (D)
- new net: D12.2 (A), D18.2 (A), D24.2 (A), D30.2 (A), D36.2 (A), D6.2 (A), Q5.3 (D)
- new net: D13.2 (A), D19.2 (A), D25.2 (A), D31.2 (A), D37.2 (A), D7.2 (A), Q6.3 (D)
- new net buzzer_drive: BZ1.2 (+), D1.2 (A), Q10.3 (D), R11.2
- new net v_bat_t: Q7.3 (D), R12.1
- no-connect marks 5 -> 8
Other:
- moved on the sheet: BT1, BT2, C1, C2, C3, C4, C5, C6, C7, C8, J1, L1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

Commit message: Add pcb rev2
also design planetary gears for mechanics and make sure they fit
Connections:
- net led_a0: now also U2.27 (PB7); no longer U2.23 (PB3)
- net led_a1: now also U2.26 (PB6); no longer U2.24 (PB4)
- net led_a3: now also U2.24 (PB4); no longer U2.26 (PB6)
- net led_a4: now also U2.23 (PB3); no longer U2.27 (PB7)
- net led_c0: now also R6.1; no longer R1.1
- net led_c1: now also R7.1; no longer R3.1
- net led_c2: now also R8.1; no longer R5.1
- net led_c3: now also R1.1; no longer R6.1
- net led_c4: now also R3.1; no longer R7.1
- net led_c5: now also R5.1; no longer R8.1
- no-connect marks 8 -> 7
Changed lines of the file:
@@
 	-1   0    0    1
 $EndComp
-Text GLabel 6800 4600 0    50   Input ~ 0
+Text GLabel 6850 4600 1    50   Input ~ 0
 vcc
-Wire Wire Line
-	6800 4600 6850 4600
 Wire Wire Line
 	6850 4600 6850 4700
@@
 Text GLabel 10200 5850 2    50   Input ~ 0
 led_a5
-Text GLabel 10200 5750 2    50   Input ~ 0
+Text GLabel 10200 5350 2    50   Input ~ 0
 led_a4
-Text GLabel 10200 5650 2    50   Input ~ 0
+Text GLabel 10200 5450 2    50   Input ~ 0
 led_a3
 Text GLabel 10200 5550 2    50   Input ~ 0
 led_a2
-Text GLabel 10200 5450 2    50   Input ~ 0
+Text GLabel 10200 5650 2    50   Input ~ 0
 led_a1
-Text GLabel 10200 5350 2    50   Input ~ 0
+Text GLabel 10200 5750 2    50   Input ~ 0
 led_a0
 NoConn ~ 10200 5250
@@
 	7550 2600 7800 2600
 Connection ~ 7800 2600
-Text GLabel 6150 4950 3    50   Input ~ 0
+Text GLabel 3550 4950 3    50   Input ~ 0
 led_c5
 $Comp
@@
 	6150 4700 6150 4650
 Connection ~ 6150 4650
-Text GLabel 5250 4950 3    50   Input ~ 0
+Text GLabel 2700 4950 3    50   Input ~ 0
 led_c4
 $Comp
@@
 Wire Wire Line
 	5250 4700 5250 4650
-Text GLabel 4450 4950 3    50   Input ~ 0
+Text GLabel 1850 4950 3    50   Input ~ 0
 led_c3
 $Comp
@@
 Wire Wire Line
 	4450 4700 4450 4650
-Text GLabel 3550 4950 3    50   Input ~ 0
+Text GLabel 6150 4950 3    50   Input ~ 0
 led_c2
 $Comp
@@
 Wire Wire Line
 	3550 4700 3550 4650
-Text GLabel 2700 4950 3    50   Input ~ 0
+Text GLabel 5250 4950 3    50   Input ~ 0
 led_c1
 $Comp
@@
 Wire Wire Line
 	2700 4700 2700 4650
-Text GLabel 1850 4950 3    50   Input ~ 0
+Text GLabel 4450 4950 3    50   Input ~ 0
 led_c0
 $Comp
@@
 $EndComp
 Connection ~ 10200 2650
-NoConn ~ 7000 4700
 Text Label 8800 2800 0    50   ~ 0
 buzzer_drive
